File: diy-ecg-pcb-uno.kicad_pcb (KiCad board)
At the start: 2 copper layers, 53.3 x 68.6 mm, 31 parts, among them J1 ECG_Cable, J2 RC, J3 LC, J4 Analog, J5 Digital_08, J6 Power, J7 Digital_10, J8 VG, J9 CM, U1 MCP6004

Commit message: Initial Project Upload
Parts:
- renumbered PPG to J10
Connections:
- J7 pad 3: unconnected-(J7-AREF-Pad3) -> Bat+
Routing:
- net Bat+: track 128.4 -> 136.3 mm
Other:
- board text added: "AREF"
