File: diy-ecg-pcb-uno.kicad_sch (KiCad schematic)
At the start: 29 parts, among them J1 ECG_Cable, J10 PPG, J2 RC, J3 LC, J4 Analog, J5 Digital_08, J6 Power, J7 Digital_10, J8 VG, J9 CM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

Commit message: Initial Project Upload
Connections:
- net Bat+: now also J7.3 (AREF)
Changed lines of the file:
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@@
+		)
+	)
+	(global_label "Bat+"
+		(shape input)
+		(at 208.28 107.95 180)
+		(fields_autoplaced yes)
+		(effects
+			(font
+				(size 1.27 1.27)
+			)
+			(justify right)
+		)
+		(property "Intersheetrefs" "${INTERSHEET_REFS}"
+			(at 200.5777 107.95 0)
+			(effects
+				(font
+					(size 1.27 1.27)
+				)
+				(justify right)
+				(hide yes)
+			)
 		)
 	)
